File: gillen.kicad_pcb (KiCad board)
At the start: 2 copper layers, 34 x 25 mm, 31 parts, among them J1 4-6V, J2 Battery, J3 USB, J4 USBOUT, J5 DCOUT, Q1 SI2307, U1 TP5410, U2 ME6211

Commit message: Address DRC and tidy up assembly info
Parts:
- D1: value DC IN -> WHITE
- D3: value STBY -> GREEN
- D4: value CHG -> RED
- D5: value 3A20V -> B340A
Other:
- board size 34 x 25 mm -> 30 x 25 mm
- board text added: "VBUS D- D+ GND GND"
- board text removed: "VBUS D+ D- GND GND"
