File: gillen.kicad_sch (KiCad schematic)
At the start: 31 parts, among them J1 4-6V, J2 Battery, J3 USB, J4 USBOUT, J5 DCOUT, Q1 SI2307, U1 TP5410, U2 ME6211

Commit message: Address DRC and tidy up assembly info
Parts:
- D1: value DC IN -> WHITE
- D3: value STBY -> GREEN
- D4: value CHG -> RED
- D5: value 3A20V -> B340A
Other:
- note added: "1.2"
- note added: "Errata 1v0 - micro USB pins were reversed 1v1 - usb d-/d+ reversed on output header silkscreen"
Changed lines of the file:
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@@
     (effects (font (size 3.5 3.5) (thickness 0.7) bold) (justify left bottom))
+  )
+  (text "Errata\n1v0 - micro USB pins were reversed\n1v1 - usb d-/d+ reversed on output header silkscreen"
+    (at 300.99 170.18 0)
+    (effects (font (size 1.27 1.27)) (justify left bottom))
+  )
+  (text "1.2" (at 269.24 194.31 0)
+    (effects (font (size 1.27 1.27)) (justify left bottom))
   )
   (text "C9 close to regulator.\nC10,11 close to load." (at 232.41 93.98 0)
@@
     (in_bom yes) (on_board yes)
     (property "Reference" "D1" (id 0) (at 115.57 124.46 0))
-    (property "Value" "DC IN" (id 1) (at 115.57 130.81 0))
+    (property "Value" "WHITE" (id 1) (at 115.57 130.81 0))
     (property "Footprint" "LED_SMD:LED_0603_1608Metric" (id 2) (at 111.76 124.46 0)
       (effects (font (size 1.27 1.27)) hide)
@@
       (effects (font (size 1.27 1.27)) (justify right))
     )
-    (property "Value" "CHG" (id 1) (at 144.78 101.6 90)
+    (property "Value" "RED" (id 1) (at 144.78 101.6 90)
       (effects (font (size 1.27 1.27)) (justify right))
     )
@@
       (effects (font (size 1.27 1.27)) (justify right))
     )
-    (property "Value" "STBY" (id 1) (at 131.445 100.965 90)
+    (property "Value" "GREEN" (id 1) (at 131.445 100.965 90)
       (effects (font (size 1.27 1.27)) (justify right))
     )
@@
     (in_bom yes) (on_board yes)
     (property "Reference" "D5" (id 0) (at 157.48 96.52 0))
-    (property "Value" "3A20V" (id 1) (at 166.37 96.52 0))
+    (property "Value" "B340A" (id 1) (at 166.37 96.52 0))
     (property "Footprint" "Diode_SMD:D_SMB" (id 2) (at 161.29 97.79 90)
       (effects (font (size 1.27 1.27)) hide)
@@
     )
     (path "/00000000-0000-0000-0000-00005db297b1"
-      (reference "D1") (unit 1) (value "DC IN") (footprint "LED_SMD:LED_0603_1608Metric")
+      (reference "D1") (unit 1) (value "WHITE") (footprint "LED_SMD:LED_0603_1608Metric")
     )
     (path "/91ac6868-ff9a-4c8f-aa54-f2f9e443f32b"
@@
     )
     (path "/00000000-0000-0000-0000-000061c7f546"
-      (reference "D3") (unit 1) (value "STBY") (footprint "LED_SMD:LED_0603_1608Metric")
+      (reference "D3") (unit 1) (value "GREEN") (footprint "LED_SMD:LED_0603_1608Metric")
     )
     (path "/00000000-0000-0000-0000-000061850c19"
-      (reference "D4") (unit 1) (value "CHG") (footprint "LED_SMD:LED_0603_1608Metric")
+      (reference "D4") (unit 1) (value "RED") (footprint "LED_SMD:LED_0603_1608Metric")
     )
     (path "/00000000-0000-0000-0000-000061ca88bd"
-      (reference "D5") (unit 1) (value "3A20V") (footprint "Diode_SMD:D_SMB")
+      (reference "D5") (unit 1) (value "B340A") (footprint "Diode_SMD:D_SMB")
     )
     (path "/dfe5e1e0-243a-4be9-847f-2113b384867b"
